Commit message: created launch file to upload urdf model to rviz.

File: src/bumperbot_description/urdf/bumperbot.urdf.xacro (robot description, xacro)
@@ -1,77 +1,77 @@
 <?xml version="1.0"?>
 <robot xmlns:xacro="http://www.ros.org/wiki/xacro" name="bumperbot">
-  <!-- Base Footprint -->
-  <link name="base_footprint"/>
-  <!-- Base Link -->
-  <link name="base_link">
-    <visual>
-      <origin rpy="0 0 0" xyz="0 0 0"/>
-      <geometry>
-        <!-- Option 1: Use a simple box if you don't have a mesh -->
-        <!-- <box size="0.3 0.2 0.1"/> -->
-        <!-- Option 2: Use your mesh if it exists -->
-        <mesh filename="package://bumperbot_description/meshes/base_link.STL"/>
-      </geometry>
-    </visual>
-  </link>
-  <!-- Joint between base_footprint and base_link -->
-  <joint name="base_joint" type="fixed">
-    <parent link="base_footprint"/>
-    <child link="base_link"/>
-    <origin xyz="0 0 0.033" rpy="0 0 0"/>
-  </joint>
-  <link name="wheel_right_link">
-    <visual>
-      <origin rpy ="1.57 0 0" xyz ="0 0 0"/>
-      <geometry>
-        <mesh filename="package://bumperbot_description/meshes/wheel_right_link.STL"/>
-      </geometry>
-    </visual>
-  </link>
-  <joint name="wheel_right_joint" type="continuous">
-    <parent link="base_link"/>
-    <child link="wheel_right_link"/>
-    <axis xyz ="0 1 0"/>
-    <origin xyz="0 -0.07 0" rpy="0 0 0"/>
-  </joint>
-  <link name="wheel_left_link">
-    <visual>
-      <origin rpy ="-1.57 0 0" xyz ="0 0 0"/>
-      <geometry>
-        <mesh filename="package://bumperbot_description/meshes/wheel_left_link.STL"/>
-      </geometry>
-    </visual>
-  </link>
-  <joint name="wheel_left_joint" type="continuous">
-    <parent link="base_link"/>
-    <child link="wheel_left_link"/>
-    <axis xyz ="0 1 0"/>
-    <origin xyz="0 0.07 0" rpy="0 0 0"/>
-  </joint>
-  <link name="caster_front_link">
-    <visual>
-      <origin rpy="0 0 0" xyz = "0 0 0"/>
-      <geometry>
-        <mesh filename="package://bumperbot_description/meshes/caster_front_link.STL"/>
-      </geometry>
-    </visual>
-  </link>
-  <joint name="caster_front_link" type="continuous">
-    <parent link="base_link"/>
-    <child link="caster_front_link"/>
-    <origin rpy="0 0 0" xyz="0.04755 0 -0.0275"/>
-  </joint>
-  <link name="caster_rear_link">
-    <visual>
-      <origin rpy="0 0 0" xyz = "0 0 0"/>
-      <geometry>
-        <mesh filename="package://bumperbot_description/meshes/caster_rear_link.STL"/>
-      </geometry>
-    </visual>
-  </link>
-  <joint name="caster_rear_link" type="continuous">
-    <parent link="base_link"/>
-    <child link="caster_rear_link"/>
-    <origin rpy="0 0 0" xyz="-0.04755 0 0.0275"/>
-  </joint>
+    <link name="base_footprint"/>
+    <link name="base_link">
+        <visual>
+            <origin rpy="0 0 0" xyz="0 0 0"/>
+            <geometry>
+                <mesh filename="package://bumperbot_description/meshes/base_link.STL"/>
+            </geometry>
+        </visual>
+        <collision>
+            <origin rpy="0 0 0" xyz="0 0 0"/>
+            <geometry>
+                <mesh filename="package://bumperbot_description/meshes/base_link.STL"/>
+            </geometry>
+        </collision>
+    </link>
+    <joint name="base_joint" type="fixed">
+        <parent link="base_footprint"/>
+        <child link="base_link"/>
+        <origin xyz="0 0 0.033" rpy="0 0 0"/>
+    </joint>
+    <link name="wheel_right_link">
+        <visual>
+            <origin xyz="0 0 0" rpy="1.57 0 0"/>
+            <geometry>
+                <mesh filename="package://bumperbot_description/meshes/wheel_right_link.STL"/>
+            </geometry>
+        </visual>
+    </link>
+    <joint name="wheel_right_joint" type="continuous">
+        <origin xyz="0 -0.07 0" rpy="0 0 0"/>
+        <parent link="base_link"/>
+        <child link="wheel_right_link"/>
+        <axis xyz="0 1 0"/>
+    </joint>
+    <link name="wheel_left_link">
+        <visual>
+            <origin xyz="0 0 0" rpy="-1.57 0 0"/>
+            <geometry>
+                <mesh filename="package://bumperbot_description/meshes/wheel_left_link.STL"/>
+            </geometry>
+        </visual>
+    </link>
+    <joint name="wheel_left_joint" type="continuous">
+        <origin xyz="0 0.07 0" rpy="0 0 0"/>
+        <parent link="base_link"/>
+        <child link="wheel_left_link"/>
+        <axis xyz="0 1 0"/>
+    </joint>
+    <link name="caster_front_link">
+        <visual>
+            <origin xyz="0.0 0.0 0.0" rpy="0.0 0.0 0.0"/>
+            <geometry>
+                <mesh filename="package://bumperbot_description/meshes/caster_front_link.STL"/>
+            </geometry>
+        </visual>
+    </link>
+    <joint name="caster_front_joint" type="fixed">
+        <origin xyz="0.04755 0 -0.0275" rpy="0 0 0"/>
+        <parent link="base_link"/>
+        <child link="caster_front_link"/>
+    </joint>
+    <link name="caster_rear_link">
+        <visual>
+            <origin xyz="0.0 0.0 0.0" rpy="0.0 0.0 0.0"/>
+            <geometry>
+                <mesh filename="package://bumperbot_description/meshes/caster_rear_link.STL"/>
+            </geometry>
+        </visual>
+    </link>
+    <joint name="caster_rear_joint" type="fixed">
+        <origin xyz="-0.04755 0 -0.0275" rpy="0 0 0"/>
+        <parent link="base_link"/>
+        <child link="caster_rear_link"/>
+    </joint>
 </robot>

Commit message: Fixed urdf  errors.

File: src/bumperbot_description/urdf/bumperbot.urdf.xacro (robot description, xacro)
@@ -1,10 +1,33 @@
 <?xml version="1.0"?>
 <robot xmlns:xacro="http://www.ros.org/wiki/xacro" name="bumperbot">
-    <link name="base_footprint"/>
+    <xacro:include filename="$(find bumperbot_description)/urdf/bumperbot_gazebo.xacro"/>
+    <xacro:include filename="$(find bumperbot_description)/urdf/bumperbot_ros2_control.xacro"/>
+    <link name="base_footprint">
+        <inertial>
+            <mass value="0.001"/>
+            <inertia
+                ixx="0.000001"
+                ixy="0.0"
+                ixz="0.0"
+                iyy="0.000001"
+                iyz="0.0"
+                izz="0.000001"/>
+        </inertial>
+    </link>
     <link name="base_link">
+        <inertial>
+            <mass value="1.0"/>
+            <inertia
+                ixx="0.001"
+                ixy="0.0"
+                ixz="0.0"
+                iyy="0.001"
+                iyz="0.0"
+                izz="0.001"/>
+        </inertial>
         <visual>
             <origin rpy="0 0 0" xyz="0 0 0"/>
             <geometry>
-                <mesh filename="package://bumperbot_description/meshes/base_link.STL"/>
+                <mesh filename="file://$(find bumperbot_description)/meshes/base_link.STL"/>
             </geometry>
         </visual>
@@ -12,5 +35,5 @@
             <origin rpy="0 0 0" xyz="0 0 0"/>
             <geometry>
-                <mesh filename="package://bumperbot_description/meshes/base_link.STL"/>
+                <box size="0.12 0.10 0.08"/>
             </geometry>
         </collision>
@@ -22,10 +45,27 @@
     </joint>
     <link name="wheel_right_link">
+        <!-- Added for Gazebo diagnostic -->
+        <inertial>
+            <mass value="0.1"/>
+            <inertia
+                ixx="0.0001"
+                ixy="0.0"
+                ixz="0.0"
+                iyy="0.0001"
+                iyz="0.0"
+                izz="0.0001"/>
+        </inertial>
         <visual>
-            <origin xyz="0 0 0" rpy="1.57 0 0"/>
+            <origin rpy="1.57 0 0" xyz="0 0.015 0"/>
             <geometry>
-                <mesh filename="package://bumperbot_description/meshes/wheel_right_link.STL"/>
+                <mesh filename="file://$(find bumperbot_description)/meshes/wheel_right_link.STL"/>
             </geometry>
         </visual>
+        <collision>
+            <origin rpy="1.57 0 0" xyz="0 -0.015 0"/>
+            <geometry>
+                <sphere radius="0.033"/>
+            </geometry>
+        </collision>
     </link>
     <joint name="wheel_right_joint" type="continuous">
@@ -36,10 +76,26 @@
     </joint>
     <link name="wheel_left_link">
+        <inertial>
+            <mass value="0.1"/>
+            <inertia
+                ixx="0.0001"
+                ixy="0.0"
+                ixz="0.0"
+                iyy="0.0001"
+                iyz="0.0"
+                izz="0.0001"/>
+        </inertial>
         <visual>
-            <origin xyz="0 0 0" rpy="-1.57 0 0"/>
+            <origin rpy="1.57 0 0" xyz="0 0.015 0"/>
             <geometry>
-                <mesh filename="package://bumperbot_description/meshes/wheel_left_link.STL"/>
+                <mesh filename="file://$(find bumperbot_description)/meshes/wheel_left_link.STL"/>
             </geometry>
         </visual>
+        <collision>
+            <origin rpy="1.57 0 0" xyz="0 0.015 0"/>
+            <geometry>
+                <sphere radius="0.033"/>
+            </geometry>
+        </collision>
     </link>
     <joint name="wheel_left_joint" type="continuous">
@@ -51,9 +107,15 @@
     <link name="caster_front_link">
         <visual>
-            <origin xyz="0.0 0.0 0.0" rpy="0.0 0.0 0.0"/>
+            <origin xyz="0 0 0" rpy="0 0 0"/>
             <geometry>
-                <mesh filename="package://bumperbot_description/meshes/caster_front_link.STL"/>
+                <mesh filename="file://$(find bumperbot_description)/meshes/caster_front_link.STL"/>
             </geometry>
         </visual>
+        <collision>
+            <origin rpy="0 0 0" xyz="0 0 0"/>
+            <geometry>
+                <sphere radius="0.005"/>
+            </geometry>
+        </collision>
     </link>
     <joint name="caster_front_joint" type="fixed">
@@ -64,9 +126,15 @@
     <link name="caster_rear_link">
         <visual>
-            <origin xyz="0.0 0.0 0.0" rpy="0.0 0.0 0.0"/>
+            <origin xyz="0 0 0" rpy="0 0 0"/>
             <geometry>
-                <mesh filename="package://bumperbot_description/meshes/caster_rear_link.STL"/>
+                <mesh filename="file://$(find bumperbot_description)/meshes/caster_rear_link.STL"/>
             </geometry>
         </visual>
+        <collision>
+            <origin rpy="0 0 0" xyz="0 0 0"/>
+            <geometry>
+                <sphere radius="0.005"/>
+            </geometry>
+        </collision>
     </link>
     <joint name="caster_rear_joint" type="fixed">

Commit message: Now the bot is controlled through controller package of ros2.

File: src/bumperbot_description/urdf/bumperbot.urdf.xacro (robot description, xacro)
@@ -35,5 +35,5 @@
             <origin rpy="0 0 0" xyz="0 0 0"/>
             <geometry>
-                <box size="0.12 0.10 0.08"/>
+                <box size="0.12 0.10 0.06"/>
             </geometry>
         </collision>
@@ -63,7 +63,7 @@
         </visual>
         <collision>
-            <origin rpy="1.57 0 0" xyz="0 -0.015 0"/>
+            <origin rpy="1.57 0 0" xyz="0 0 0"/>
             <geometry>
-                <sphere radius="0.033"/>
+                <cylinder radius="0.033" length="0.03"/>
             </geometry>
         </collision>
@@ -93,7 +93,7 @@
         </visual>
         <collision>
-            <origin rpy="1.57 0 0" xyz="0 0.015 0"/>
+            <origin rpy="1.57 0 0" xyz="0 0 0"/>
             <geometry>
-                <sphere radius="0.033"/>
+                <cylinder radius="0.033" length="0.03"/>
             </geometry>
         </collision>

File: src/bumperbot_description/urdf/bumperbot_gazebo.xacro (robot description, xacro)
@@ -1,5 +1,5 @@
 <?xml version="1.0"?>
 <robot name="bumperbot" xmlns:xacro="http://www.ros.org/wiki/xacro">
-    <!-- <transmission name="wheel_right_transmission">
+    <transmission name="wheel_right_transmission">
         <plugin>transmission_interface/SimpleTransmission</plugin>
         <type>transmission_interface/SimpleTransmission</type>
@@ -8,6 +8,6 @@
         </joint>
         <actuator name="wheel_right_motor" role="actuator_right"/>
-    </transmission> -->
-    <!-- <transmission name="wheel_left_transmission">
+    </transmission>
+    <transmission name="wheel_left_transmission">
         <plugin>transmission_interface/SimpleTransmission</plugin>
         <type>transmission_interface/SimpleTransmission</type>
@@ -16,5 +16,5 @@
         </joint>
         <actuator name="wheel_left_motor" role="actuator_left"/>
-    </transmission> -->
+    </transmission>
     <gazebo reference="wheel_right_link">
         <mu1>1.0</mu1>
@@ -49,5 +49,5 @@
         <maxVel>0.1</maxVel>
     </gazebo>
-    <!-- <gazebo>
+    <gazebo>
         <plugin filename="libgazebo_ros2_control.so" name="gazebo_ros2_control">
             <robot_param>robot_description</robot_param>
@@ -55,4 +55,4 @@
             <parameters>$(find bumperbot_controller)/config/bumperbot_controllers.yaml</parameters>
         </plugin>
-    </gazebo> -->
+    </gazebo>
 </robot>
